File: kicad/helios.kicad_pcb (KiCad board)
At the start: 2 copper layers, 65 x 56 mm, 5 parts, among them J2 RPi_GPIO

Commit message: Began board layout
Parts:
- removed ? (x4): , RPi_Hat:RPi_Hat_Mounting_Hole
- added 111: XT30, helios_kicad_lib:XT30P, F.Cu at (121.5, 114.0)
- added C1: 0.1uF, Capacitor_SMD:C_0402_1005Metric, F.Cu at (131.7, 102.9)
- added C10: 0.1uF, Capacitor_SMD:C_0402_1005Metric, F.Cu at (159.9, 95.8)
- added C11: 0.1uF, Capacitor_SMD:C_0402_1005Metric, F.Cu at (157.3, 97.4)
- added C12: 10uF, Capacitor_SMD:C_0402_1005Metric, F.Cu at (138.0, 97.1)
- added C13: 1uF, Capacitor_SMD:C_0402_1005Metric, F.Cu at (151.1, 86.4)
- added C14: 0.1uF, Capacitor_SMD:C_0402_1005Metric, F.Cu at (161.7, 88.4)
- added C15: 0.1uF, Capacitor_SMD:C_0402_1005Metric, F.Cu at (142.4, 87.1)
- added C16: 0.1uF, Capacitor_SMD:C_0402_1005Metric, F.Cu at (141.8, 95.5)
- added C17: 0.1uF, Capacitor_SMD:C_0402_1005Metric, F.Cu at (131.3, 88.4)
- added C18: 10uF, Capacitor_SMD:C_0402_1005Metric, F.Cu at (132.7, 86.5)
- added C19: 0.1uF 50V, Capacitor_SMD:C_1206_3216Metric, F.Cu at (126.5, 108.4)
- added C2: 0.1uF, Capacitor_SMD:C_0402_1005Metric, F.Cu at (149.4, 110.1)
- added C20: 0.1uF 50V, Capacitor_SMD:C_1206_3216Metric, F.Cu at (121.6, 108.4)
- added C21: 0.1uF 50V, Capacitor_SMD:C_1206_3216Metric, F.Cu at (124.1, 108.4)
- added C22: 0.1uF 50V, Capacitor_SMD:C_1206_3216Metric, F.Cu at (126.1, 92.7)
- added C23: 0.01uF, Capacitor_SMD:C_0402_1005Metric, F.Cu at (127.7, 105.3)
- added C24: 10uF, Capacitor_SMD:C_1206_3216Metric, F.Cu at (130.9, 96.6)
- added C25: 22uF 16V, Capacitor_SMD:C_0603_1608Metric, F.Cu at (129.1, 91.4)
- added C26: 22uF 16V, Capacitor_SMD:C_0603_1608Metric, F.Cu at (129.1, 89.8)
- added C3: 0.1uF, Capacitor_SMD:C_0402_1005Metric, F.Cu at (131.2, 90.5)
- added C4: 0.1uF, Capacitor_SMD:C_0402_1005Metric, F.Cu at (149.5, 91.8)
- added C5: 0.1uF, Capacitor_SMD:C_0402_1005Metric, F.Cu at (131.4, 109.5)
- added C6: 0.1uF, Capacitor_SMD:C_0402_1005Metric, F.Cu at (152.0, 103.2)
- added C7: 1uF, Capacitor_SMD:C_0402_1005Metric, F.Cu at (150.6, 87.4)
- added C8: 0.1uF, Capacitor_SMD:C_0402_1005Metric, F.Cu at (132.7, 87.3)
- added C9: 0.1uF, Capacitor_SMD:C_0402_1005Metric, F.Cu at (149.4, 89.7)
- added D1: Blue, LED_SMD:LED_0603_1608Metric, F.Cu at (134.0, 116.7)
- added D2: Blue, LED_SMD:LED_0603_1608Metric, F.Cu at (134.3, 114.8)
- added D3: Red, LED_SMD:LED_0603_1608Metric, F.Cu at (145.7, 87.9)
- added D4: Blue, LED_SMD:LED_0603_1608Metric, F.Cu at (164.9, 81.7)
- added D5: Blue, LED_SMD:LED_0603_1608Metric, F.Cu at (165.0, 83.9)
- added D6: Red, LED_SMD:LED_0603_1608Metric, F.Cu at (167.2, 85.9)
- added D7: SMF48A-E3-08, helios_kicad_lib:SMF, F.Cu at (129.5, 106.3)
- added D8: Red, LED_SMD:LED_0603_1608Metric, F.Cu at (128.4, 84.6)
- added F1: 0686F4000-01, Fuse:Fuse_0603_1608Metric, F.Cu at (129.3, 112.5)
- added H1: MountingHole_Pad, MountingHole:MountingHole_2.7mm_M2.5_DIN965, F.Cu at (118.8, 77.3)
- added H2: MountingHole_Pad, MountingHole:MountingHole_2.7mm_M2.5_DIN965, F.Cu at (118.8, 126.3)
- added H3: MountingHole_Pad, MountingHole:MountingHole_2.7mm_M2.5_DIN965, F.Cu at (176.8, 126.3)
- added H4: MountingHole_Pad, MountingHole:MountingHole_2.7mm_M2.5_DIN965, F.Cu at (176.8, 77.3)
- added J1: CAN 1 Conn, Connector_JST:JST_PH_B3B-PH-K_1x03_P2.00mm_Vertical, F.Cu at (144.0, 113.6)
- added J14: Serial Breakout, Connector_PinHeader_2.54mm:PinHeader_1x03_P2.54mm_Vertical, F.Cu at (128.7, 57.6)
- added J19: Raspberry_Pi_4, helios_kicad_lib:Pin_Header_Straight_2x20, F.Cu at (147.8, 77.3)
- added J22: I2C Breakout, Connector_PinHeader_2.54mm:PinHeader_1x03_P2.54mm_Vertical, F.Cu at (131.4, 120.9)
- added J25: Stemma QT, helios_kicad_lib:JST_SH4, F.Cu at (127.6, 127.2)
- added J26: Stemma QT, helios_kicad_lib:JST_SH4, F.Cu at (134.9, 127.2)
- added J3: CAN 2 Conn, Connector_JST:JST_PH_B3B-PH-K_1x03_P2.00mm_Vertical, F.Cu at (144.2, 102.6)
- added J4: CAN 4 Conn, Connector_JST:JST_PH_B3B-PH-K_1x03_P2.00mm_Vertical, F.Cu at (164.2, 104.2)
- added J5: SWD Programming, Connector_JST:JST_PH_B6B-PH-K_1x06_P2.00mm_Vertical, F.Cu at (149.9, 82.4)
- added J6: SWD Programming, Connector_JST:JST_PH_B6B-PH-K_1x06_P2.00mm_Vertical, F.Cu at (131.9, 82.5)
- added J7: USB_B_Micro, Connector_USB:USB_Micro-AB_Molex_47590-0001, F.Cu at (154.1, 128.3)
- added J8: USB_B_Micro, Connector_USB:USB_Micro-AB_Molex_47590-0001, F.Cu at (143.7, 128.3)
- added JP1: Servo Breakout 1, helios_kicad_lib:3X04, F.Cu at (175.6, 89.4)
- added JP2: Servo Breakout 2, helios_kicad_lib:3X04, F.Cu at (175.4, 111.7)
- added JP3: Servo Breakout 3, helios_kicad_lib:3X04, F.Cu at (175.4, 100.6)
- added L1: 10uH, helios_kicad_lib:IND_YUDEN_NS10165_YDN, F.Cu at (121.0, 85.9)
- added R1: 120, Resistor_SMD:R_0402_1005Metric, F.Cu at (140.6, 109.6)
- added R10: 220, Resistor_SMD:R_0402_1005Metric, F.Cu at (164.2, 85.9)
- added R11: 105k, Resistor_SMD:R_0402_1005Metric, F.Cu at (128.6, 101.7)
- added R12: 560, Resistor_SMD:R_0402_1005Metric, F.Cu at (128.4, 81.7)
- added R13: 22.1k, Resistor_SMD:R_0402_1005Metric, F.Cu at (128.6, 100.5)
- added R2: 120, Resistor_SMD:R_0402_1005Metric, F.Cu at (158.3, 110.3)
- added R3: 120, Resistor_SMD:R_0402_1005Metric, F.Cu at (140.7, 102.8)
- added R4: 120, Resistor_SMD:R_0402_1005Metric, F.Cu at (161.0, 103.0)
- added R5: 220, Resistor_SMD:R_0402_1005Metric, F.Cu at (131.6, 116.5)
- added R6: 220, Resistor_SMD:R_0402_1005Metric, F.Cu at (131.5, 114.7)
- added R7: 220, Resistor_SMD:R_0402_1005Metric, F.Cu at (145.7, 90.8)
- added R8: 220, Resistor_SMD:R_0402_1005Metric, F.Cu at (168.1, 81.7)
- added R9: 220, Resistor_SMD:R_0402_1005Metric, F.Cu at (168.2, 83.7)
- added U1: STM32G474CET6, helios_kicad_lib:STM32G474CET6, F.Cu at (137.4, 91.0)
- added U10: BNO055, BNO055_STEMMA_QT:BNO055, F.Cu at (77.3, 73.9)
- added U11: XT30, helios_kicad_lib:XT30P, F.Cu at (174.3, 120.8)
- added U12: MAX17504ATP+T, helios_kicad_lib:MAX17504ATP&plus_T, F.Cu at (124.3, 99.7)
- added U2: TCAN334G, helios_kicad_lib:TCAN334G, F.Cu at (135.9, 109.6)
- added U3: TCAN334G, helios_kicad_lib:TCAN334G, F.Cu at (154.0, 110.2)
- added U4: TCAN334G, helios_kicad_lib:TCAN334G, F.Cu at (136.1, 102.9)
- added U5: TCAN334G, helios_kicad_lib:TCAN334G, F.Cu at (156.4, 103.2)
- added U6: STM32G474CET6, helios_kicad_lib:STM32G474CET6, F.Cu at (155.6, 91.3)
- added U7: USBLC6-2SC6, Package_TO_SOT_SMD:SOT-23-6, F.Cu at (154.1, 122.2)
- added U8: USBLC6-2SC6, Package_TO_SOT_SMD:SOT-23-6, F.Cu at (143.7, 122.2)
- added U9: XT30, helios_kicad_lib:XT30P, F.Cu at (121.4, 119.8)
- J2: value RPi_GPIO -> CAN 3 Conn; footprint RPi_Hat:Pin_Header_Straight_2x20 -> Connector_JST:JST_PH_B3B-PH-K_1x03_P2.00mm_Vertical
- moved J2 37.1 mm to (160.4, 112.1)
Connections:
- J2 pad 1: (no net) -> Net-(J2-Pad1)
- J2 pad 2: (no net) -> Net-(J2-Pad2)
- J2 pad 3: (no net) -> GND

Commit message: About to start routing
Parts:
- moved U10 87.8 mm to (161.1, 100.2)
- moved J14 29.9 mm to (132.5, 87.3), turned to 180 degrees
- moved J4 20.5 mm to (147.9, 116.6), turned to 180 degrees
- moved J3 15.0 mm to (138.9, 116.6), turned to 180 degrees
- moved J2 12.6 mm to (147.9, 111.0), turned to 180 degrees
- moved C5 12.0 mm to (135.8, 98.4), turned to 180 degrees
- moved C2 12.0 mm to (146.9, 98.4), turned to 180 degrees
- moved R2 11.8 mm to (146.9, 107.0), turned to 180 degrees
- moved C1 10.7 mm to (141.4, 98.4), turned to 180 degrees
- moved U3 10.3 mm to (146.9, 102.7), turned to 270 degrees
- moved R9 9.28 mm to (177.5, 82.8)
- moved D5 9.28 mm to (174.2, 83.0)
- moved D4 9.26 mm to (174.2, 81.3)
- moved R8 9.26 mm to (177.3, 81.4)
- moved C6 8.01 mm to (158.6, 98.8), turned to 180 degrees
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Routing:
- added copper zone on In2.Cu-3V3, net +3V3
- added copper zone on In1.Cu-GND, net GND
Other:
- copper layers 2 -> 4

Commit message: Finished routing
Parts:
- added J9: Power Breakout, helios_kicad_lib:Eagle_1X03, F.Cu at (126.0, 126.2)
- H1, H2, H3, H4: footprint MountingHole:MountingHole_2.7mm_M2.5_DIN965 -> MountingHole:MountingHole_2.7mm_M2.5_DIN965_Pad
- J14: footprint Connector_PinHeader_2.54mm:PinHeader_1x03_P2.54mm_Vertical -> helios_kicad_lib:Eagle_1X03
- J22: footprint Connector_PinHeader_2.54mm:PinHeader_1x03_P2.54mm_Vertical -> Connector_PinHeader_2.54mm:PinHeader_1x04_P2.54mm_Vertical
- moved C17 31.1 mm to (167.4, 90.6), turned to 0 degrees
- moved C18 29.2 mm to (166.9, 89.1), turned to 90 degrees
- moved D1 27.6 mm to (134.7, 90.4), turned to 90 degrees
- moved R9 27.2 mm to (151.5, 90.9), turned to 270 degrees
- moved R8 26.0 mm to (153.1, 90.9), turned to 270 degrees
- moved D2 25.5 mm to (133.0, 90.4), turned to 90 degrees
- moved R5 25.3 mm to (134.7, 93.0), turned to 270 degrees
- moved D5 23.4 mm to (151.5, 88.3), turned to 90 degrees
- moved R6 23.2 mm to (133.0, 93.0), turned to 270 degrees
- moved U8 22.9 mm to (166.6, 122.3), turned to 180 degrees
- moved J8 22.9 mm to (166.6, 128.3)
- moved JP1 22.7 mm to (175.3, 112.0)
- moved JP2 22.7 mm to (175.3, 89.3)
- moved D4 22.2 mm to (153.1, 88.3), turned to 90 degrees
- moved C16 20.4 mm to (165.4, 87.2), turned to 90 degrees
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- renumbered 111 to 1111
Connections:
- net Net-(111-Pad+) renamed POWER_IN
- J6 pad 3: SWDI_2 -> SWDIO_2
- JP1 pad 4: TIM8_CH3N_1 -> TIM5_CH3_1
- JP1 pad 7: TIM20_CH1_1 -> TIM5_CH2_1
- JP2 pad 1: TIM8_CH2N_2 -> TIM20_CH1_2
- JP2 pad 10: TIM5_CH1_2 -> TIM5_CH3_2
- JP2 pad 7: TIM20_CH1_2 -> TIM8_CH2N_2
- JP3 pad 1: TIM5_CH2_1 -> TIM5_CH2_2
- JP3 pad 10: TIM5_CH3_2 -> TIM8_CH3N_1
- JP3 pad 4: TIM5_CH3_1 -> TIM5_CH1_2
- JP3 pad 7: TIM5_CH2_2 -> TIM20_CH1_1
- U1 pad 35: Net-(U1-Pad35) -> GND
- U1 pad 41: Net-(U1-Pad41) -> LED_1
- U1 pad 42: Net-(U1-Pad42) -> LED_2
- U1 pad 47: Net-(U1-Pad47) -> GND
- U1 pad 5: LED_1 -> Net-(U1-Pad5)
- U1 pad 6: LED_2 -> Net-(U1-Pad6)
- U10 pad 1: (no net) -> Net-(U10-Pad1)
- U10 pad 10: (no net) -> Net-(U10-Pad10)
- U10 pad 2: (no net) -> +3V3
- U10 pad 3: (no net) -> GND
- U10 pad 4: (no net) -> I2C2_SCL
- U10 pad 5: (no net) -> I2C2_SDA
- U10 pad 6: (no net) -> Net-(U10-Pad6)
- U10 pad 7: (no net) -> Net-(U10-Pad7)
- U10 pad 8: (no net) -> Net-(U10-Pad8)
- U10 pad 9: (no net) -> Net-(U10-Pad9)
- U6 pad 41: Net-(U6-Pad41) -> LED_3
- U6 pad 42: Net-(U6-Pad42) -> LED_4
- U6 pad 5: LED_3 -> Net-(U6-Pad5)
- U6 pad 6: LED_4 -> Net-(U6-Pad6)
Routing:
- net GND: track 0.00 -> 140.9 mm, vias 0 -> 48
- net I2C2_SDA: track 0.00 -> 138.8 mm, vias 0 -> 2
- net I2C2_SCL: track 0.00 -> 130.3 mm, vias 0 -> 3
- net +5V: track 0.00 -> 127.3 mm, vias 0 -> 8
- net +3V3: track 0.00 -> 62.1 mm, vias 0 -> 21
- net USB_D+: track 0.00 -> 49.3 mm, vias 0 -> 2
- net USB_D-: track 0.00 -> 47.9 mm, vias 0 -> 2
- net USB2_D+: track 0.00 -> 41.8 mm, vias 0 -> 2
- net USB2_D-: track 0.00 -> 41.3 mm, vias 0 -> 2
- net TIM5_CH2_1: track 0.00 -> 40.2 mm
- net TIM5_CH1_1: track 0.00 -> 38.5 mm
- net TIM5_CH3_1: track 0.00 -> 37.9 mm
- net +BATT: track 0.00 -> 35.3 mm
- net TIM8_CH2N_1: track 0.00 -> 33.4 mm
- net TIM8_CH3N_1: track 0.00 -> 33.2 mm
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- added copper zone on F.Cu, net +5V
- added copper zone on F.Cu, net GND
- added copper zone on F.Cu, net LX
- added copper zone on F.Cu, net POWER_IN
- added copper zone on F.Cu, net VIN
Other:
- outline, holes or cut-outs redrawn
- net class Default: clearance 0.2 -> 0.16; trace_width 0.25 -> 0.2
- rule trace_clearance: 0.2 -> 0.16
