File: kicad/helios.sch (KiCad schematic (older format))
At the start: 37 parts

Commit message: Added second MCU to schematic
Parts:
- added C? (x9): C_Small, symbol Device:C_Small
- added D? (x4): LED_Small, symbol Device:LED_Small
- added J?: USB_B_Micro, symbol Connector:USB_B_Micro
- added J? (x2): Conn_01x03, symbol Connector_Generic:Conn_01x03
- added J?: SWD Programming, symbol Connector_Generic:Conn_01x06
- added R? (x6): R_Small, symbol Device:R_Small
- added U? (x2): STM32G474CEU6, UFQFPN-48_7X7X0P55MM, symbol STM32G474CEU6:STM32G474CEU6
- added U?: USBLC6-2SC6, Package_TO_SOT_SMD:SOT-23-6, symbol Power_Protection:USBLC6-2SC6
- added U? (x2): TCAN334G, symbol Interface_CAN_LIN:TCAN334G
Connections:
- net +3V3: now also C?.2, C?.2, U?.3 (PC14-OSC32_IN), U?.3 (VCC), U?.3 (VCC), C?.1, C?.1, C?.1, C?.1, C?.1, C?.1, C?.2, C?.2, D?.2 (A), D?.2 (A), D?.2 (A), D?.2 (A), J?.1 (Pin_1), U?.1 (VBAT), U?.20 (VREF+), U?.21 (VDDA), U?.23 (VDD), U?.3 (PC14-OSC32_IN), U?.3 (VCC), U?.3 (VCC), U?.35 (VDD), U?.48 (VDD); no longer C?.1, C?.1
- net +5V: now also J?.1 (VBUS), U?.5 (VBUS)
- net CAN1_RX: now also U?.4 (RXD), U?.46 (PB8-BOOT0)
- net CAN1_TX: now also U?.1 (TXD), U?.47 (PB9)
- net CAN2_RX: now also U?.27 (PB14), U?.4 (RXD)
- net CAN2_TX: now also U?.1 (TXD), U?.26 (PB13)
- net GND: now also C?.1, C?.1, U?.4 (PC15-OSC32_OUT), C?.1, C?.1, C?.2, C?.2, C?.2, C?.2, C?.2, C?.2, C?.2, J?.3 (Pin_3), J?.3 (Pin_3), J?.5 (GND), J?.6 (Pin_6), U?.2 (GND), U?.2 (GND), U?.2 (GND), U?.4 (PC15-OSC32_OUT), U?.49 (EPAD), U?.5 (SHDN), U?.5 (SHDN), U?.8 (STB), U?.8 (STB)
- net NRST: now also C?.1, J?.5 (Pin_5), U?.7 (PG10-NRST)
- net SWCLK: now also J?.4 (Pin_4), U?.37 (PA14)
- net SWDIO: now also J?.3 (Pin_3), U?.36 (PA13)
- net SWO: now also J?.2 (Pin_2), U?.41 (PB3)
- net USB_CONN_D+: now also J?.3 (D+), U?.3 (I/O2)
- net USB_CONN_D-: now also J?.2 (D-), U?.1 (I/O1)
- net USB_D+: now also U?.34 (PA12), U?.4 (I/O2)
- net USB_D-: now also U?.33 (PA11), U?.6 (I/O1)
- net SPI1_NSS: now reaches U?.12 (PA4)
- net SPI1_NSS: now also U?.12 (PA4)
- net SPI1_SCK: now reaches U?.13 (PA5)
- net SPI1_SCK: now also U?.13 (PA5)
- net SPI1_MISO: now reaches U?.14 (PA6)
- net SPI1_MISO: now also U?.14 (PA6)
- net SPI1_MOSI: now reaches U?.15 (PA7)
- net SPI1_MOSI: now also U?.15 (PA7)
- net LED_1: now reaches U?.5 (PF0-OSC_IN)
- net LED_1: now also R?.2, R?.2, U?.5 (PF0-OSC_IN)
- net LED_2: now reaches U?.6 (PF1-OSC_OUT)
- net LED_2: now also R?.2, R?.2, U?.6 (PF1-OSC_OUT)
- new net: D?.1 (K), R?.1 (x4)
- new net: J?.2 (Pin_2), R?.2, U?.6 (CANL) (x2)
- new net: J?.1 (Pin_1), R?.1, U?.7 (CANH) (x2)
- no-connect marks 5 -> 53
Other:
- moved on the sheet: C?, D?, F?, J?, L?, R?, U?, U?A, U?B

Commit message: Majorly updated schematic, added footprints
Parts:
- removed C? (x9): C_Small, symbol Device:C_Small
- removed D? (x2): LED_Small, symbol Device:LED_Small
- removed J?: USB_B_Micro, symbol Connector:USB_B_Micro
- removed J? (x2): Conn_01x03, symbol Connector_Generic:Conn_01x03
- removed J?: SWD Programming, symbol Connector_Generic:Conn_01x06
- removed R? (x4): R_Small, symbol Device:R_Small
- removed U? (x4): STM32G474CEU6, UFQFPN-48_7X7X0P55MM, symbol STM32G474CEU6:STM32G474CEU6
- removed U?: USBLC6-2SC6, Package_TO_SOT_SMD:SOT-23-6, symbol Power_Protection:USBLC6-2SC6
- removed U? (x2): TCAN334G, symbol Interface_CAN_LIN:TCAN334G
- added C13: 1uF, Capacitor_SMD:C_0402_1005Metric, symbol Device:C_Small
- added C14, C15, C16, C17, C2, C4, C6: 0.1uF, Capacitor_SMD:C_0402_1005Metric, symbol Device:C_Small
- added C18: 10uF, Capacitor_SMD:C_0402_1005Metric, symbol Device:C_Small
- added D3, D6, D8: Red, LED_SMD:LED_0603_1608Metric, symbol Device:LED_Small
- added D4, D5: Blue, LED_SMD:LED_0603_1608Metric, symbol Device:LED_Small
- added J14: Serial Breakout, Connector_PinHeader_2.54mm:PinHeader_1x03_P2.54mm_Vertical, symbol Connector_Generic:Conn_01x03
- added J2: CAN 3 Conn, Connector_JST:JST_PH_B4B-PH-K_1x04_P2.00mm_Vertical, symbol Connector_Generic:Conn_01x03
- added J22: I2C Breakout, Connector_PinHeader_2.54mm:PinHeader_1x03_P2.54mm_Vertical, symbol Connector_Generic:Conn_01x04
- added J25, J26: Stemma QT, helios_kicad_lib:JST_SH4, symbol Connector_Generic:Conn_01x04
- added J4: CAN 4 Conn, Connector_JST:JST_PH_B4B-PH-K_1x04_P2.00mm_Vertical, symbol Connector_Generic:Conn_01x03
- added J6: SWD Programming, Connector_JST:JST_PH_B6B-PH-K_1x06_P2.00mm_Vertical, symbol Connector_Generic:Conn_01x06
- added J8: USB_B_Micro, Connector_USB:USB_Micro-AB_Molex_47590-0001, symbol Connector:USB_B_Micro
- added JP1: Servo Breakout 1, helios_kicad_lib:3X04, symbol header-3x04:HEADER-3X04
- added JP2: Servo Breakout 2, helios_kicad_lib:3X04, symbol header-3x04:HEADER-3X04
- added JP3: Servo Breakout 3, helios_kicad_lib:3X04, symbol header-3x04:HEADER-3X04
- added R10, R7, R8, R9: 220, Resistor_SMD:R_0402_1005Metric, symbol Device:R_Small
- added R12: 560, Resistor_SMD:R_0402_1005Metric, symbol Device:R_Small
- added R2, R4: 120, Resistor_SMD:R_0402_1005Metric, symbol Device:R_Small
- added U1, U6: STM32G474CET6, helios_kicad_lib:STM32G474CET6, symbol STM32G474CET6:STM32G474CET6
- added U10: BNO055, BNO055_STEMMA_QT:BNO055, symbol BNO055_STEMMA_QT:BNO055
- added U11: XT30, helios_kicad_lib:XT30P, symbol xt30:XT30
- added U3, U5: TCAN334G, helios_kicad_lib:TCAN334G, symbol Interface_CAN_LIN:TCAN334G
- added U8: USBLC6-2SC6, Package_TO_SOT_SMD:SOT-23-6, symbol Power_Protection:USBLC6-2SC6
- 11: renamed from ?; footprint (none) -> helios_kicad_lib:XT30P
- C1, C10, C11, C3, C5, C8, C9: renamed from C?; value C_Small -> 0.1uF; footprint (none) -> Capacitor_SMD:C_0402_1005Metric
- C12, C24: renamed from C?; value C_Small -> 10uF; footprint (none) -> Capacitor_SMD:C_0402_1005Metric
- C19, C20, C21, C22: renamed from C?; value C_Small -> 0.1uF 50V; footprint (none) -> Capacitor_SMD:C_0402_1005Metric
- C23: renamed from C?; value C_Small -> 0.01uF; footprint (none) -> Capacitor_SMD:C_0402_1005Metric
- C25, C26: renamed from C?; value C_Small -> 22uF 16V; footprint (none) -> Capacitor_SMD:C_0603_1608Metric
- C7: renamed from C?; value C_Small -> 1uF; footprint (none) -> Capacitor_SMD:C_0402_1005Metric
- D1, D2: renamed from D?; value LED_Small -> Blue; footprint (none) -> LED_SMD:LED_0603_1608Metric
- D7: renamed from D?; value D_Small -> SMF48A-E3-08; footprint (none) -> helios_kicad_lib:SMF
- F1: renamed from F?; value Fuse_Small -> 0686F4000-01; footprint (none) -> Fuse:Fuse_0603_1608Metric
- J1: renamed from J?; value Conn_01x03 -> CAN 1 Conn; footprint (none) -> Connector_JST:JST_PH_B4B-PH-K_1x04_P2.00mm_Vertical
- J19: renamed from J?; footprint (none) -> helios_kicad_lib:Pin_Header_Straight_2x20
- J3: renamed from J?; value Conn_01x03 -> CAN 2 Conn; footprint (none) -> Connector_JST:JST_PH_B4B-PH-K_1x04_P2.00mm_Vertical
- J5: renamed from J?; footprint (none) -> Connector_JST:JST_PH_B6B-PH-K_1x06_P2.00mm_Vertical
- J7: renamed from J?; footprint (none) -> Connector_USB:USB_Micro-AB_Molex_47590-0001
- L1: renamed from L?; value L_Small -> 10uH; footprint (none) -> helios_kicad_lib:IND_YUDEN_NS10165_YDN
- R1, R3: renamed from R?; value R_Small -> 120; footprint (none) -> Resistor_SMD:R_0402_1005Metric
- R11: renamed from R?; value R_Small -> 105k; footprint (none) -> Resistor_SMD:R_0402_1005Metric
- R13: renamed from R?; value R_Small -> 22.1k; footprint (none) -> Resistor_SMD:R_0402_1005Metric
- R5, R6: renamed from R?; value R_Small -> 220; footprint (none) -> Resistor_SMD:R_0402_1005Metric
- U12: renamed from U?; footprint 21-0140L_T2055-4_MXM -> helios_kicad_lib:MAX17504ATP&plus_T
- U2, U4: renamed from U?; footprint (none) -> helios_kicad_lib:TCAN334G
- U9: renamed from U?; footprint (none) -> helios_kicad_lib:XT30P
- gave numbers to parts that had none: 1
Connections:
- net +3V3: now also C13.1, C14.1, C15.1, C16.1, C17.1, C18.1, C2.2, C6.2, D3.2 (A), D4.2 (A), D5.2 (A), D6.2 (A), J22.2 (Pin_2), J25.2 (Pin_2), J26.2 (Pin_2), J6.1 (Pin_1), U1.1 (VBAT), U1.20 (VREF+), U1.21 (VDDA), U1.24 (VDD), U1.3 (PC14-OSC32_IN), U1.36 (VDD), U1.48 (VDD), U10.2 (3V3), U3.3 (VCC), U5.3 (VCC), U6.1 (VBAT), U6.20 (VREF+), U6.21 (VDDA), U6.24 (VDD), U6.3 (PC14-OSC32_IN), U6.36 (VDD), U6.48 (VDD)
- net +5V: now also D8.2 (A), J8.1 (VBUS), U8.5 (VBUS)
- net CAN1_RX: now also U1.45 (PB8-BOOT0)
- net CAN1_TX: now also U1.46 (PB9)
- net CAN2_RX: now also U1.28 (PB14)
- net CAN2_TX: now also U1.27 (PB13)
- net GND: now also C13.2, C14.2, C15.2, C16.2, C17.2, C18.2, C2.1, C4.2, C6.1, J14.1 (Pin_1), J2.3 (Pin_3), J22.1 (Pin_1), J25.1 (Pin_1), J26.1 (Pin_1), J4.3 (Pin_3), J6.6 (Pin_6), J8.5 (GND), JP1.12, JP1.3, JP1.6, JP1.9, JP2.12, JP2.3, JP2.6, JP2.9, JP3.12, JP3.3, JP3.6, JP3.9, R10.2, R12.2, R7.2, U1.19 (VSSA), U1.23 (VSS), U1.4 (PC15-OSC32_OUT), U10.3 (GND), U11.-, U3.2 (GND), U3.5 (SHDN), U3.8 (STB), U5.2 (GND), U5.5 (SHDN), U5.8 (STB), U6.19 (VSSA), U6.23 (VSS), U6.35 (VSS), U6.4 (PC15-OSC32_OUT), U6.47 (VSS), U8.2 (GND)
- net LED_1: now also U1.5 (PF0-OSC_IN)
- net LED_2: now also U1.6 (PF1-OSC_OUT)
- net NRST: now also U1.7 (PG10-NRST)
- net SPI1_MISO: now also J19.35 (GPIO19/MISO1), U6.14 (PA6)
- net SPI1_MOSI: now also J19.38 (GPIO20/MOSI1), U6.15 (PA7)
- net SPI1_NSS: now also U6.12 (PA4)
- net SPI1_SCK: now also J19.40 (GPIO21/SCLK1), U6.13 (PA5)
- net SWCLK: now also U1.38 (PA14)
- net SWDIO: now also U1.37 (PA13)
- net SWO: now also U1.40 (PB3)
- net USB_D+: now also U1.34 (PA12)
- net USB_D-: now also U1.33 (PA11)
- net at J19.10 (GPIO15/RXD): now also J14.2 (Pin_2)
- net SPI0_MOSI: now reaches J19.19 (MOSI0/GPIO10)
- net SPI0_MOSI: now also U1.15 (PA7)
- net SPI0_MISO: now reaches J19.21 (MISO0/GPIO9)
- net SPI0_MISO: now also U1.14 (PA6)
- net SPI0_SCK: now reaches J19.23 (SCLK0/GPIO11)
- net SPI0_SCK: now also U1.13 (PA5)
- net I2C2_SDA: now reaches J19.3 (SDA/GPIO2)
- net I2C2_SDA: now also J22.3 (Pin_3), J25.3 (Pin_3), J26.3 (Pin_3), U1.30 (PA8), U10.5 (SDA), U6.30 (PA8)
- net I2C2_SCL: now reaches J19.5 (SCL/GPIO3)
- net I2C2_SCL: now also J22.4 (Pin_4), J25.4 (Pin_4), J26.4 (Pin_4), U1.31 (PA9), U10.4 (SCL), U6.31 (PA9)
- net at J19.8 (GPIO14/TXD): now also J14.3 (Pin_3)
- new net: D3.1 (K), R7.1
- new net: D8.1 (K), R12.1
- new net: J2.2 (Pin_2), R2.2, U3.6 (CANL)
- new net: J2.1 (Pin_1), R2.1, U3.7 (CANH)
- new net: J4.2 (Pin_2), R4.2, U5.6 (CANL)
- new net: J4.1 (Pin_1), R4.1, U5.7 (CANH)
- new net: D4.1 (K), R8.1
- new net: D5.1 (K), R9.1
- new net: D6.1 (K), R10.1
- new net +BATT: JP1.11, JP1.2, JP1.5, JP1.8, JP2.11, JP2.2, JP2.5, JP2.8, JP3.11, JP3.2, JP3.5, JP3.8, U11.+
- new net CAN3_RX: U3.4 (RXD), U6.45 (PB8-BOOT0)
- new net CAN3_TX: U3.1 (TXD), U6.46 (PB9)
- new net CAN4_RX: U5.4 (RXD), U6.28 (PB14)
- new net CAN4_TX: U5.1 (TXD), U6.27 (PB13)
- new net LED_3: R8.2, U6.5 (PF0-OSC_IN)
- new net LED_4: R9.2, U6.6 (PF1-OSC_OUT)
- new net NRST_2: C4.1, J6.5 (Pin_5), U6.7 (PG10-NRST)
- new net SPI0_NSS: U1.12 (PA4)
- new net SWCLK_2: J6.4 (Pin_4), U6.38 (PA14)
- new net SWDIO_2: U6.37 (PA13)
- new net SWDI_2: J6.3 (Pin_3)
- new net SWO_2: J6.2 (Pin_2), U6.40 (PB3)
- new net TIM20_CH1_1: JP1.7, U1.18 (PB2)
- new net TIM20_CH1_2: JP2.7, U6.18 (PB2)
- new net TIM5_CH1_1: JP1.10, U1.8 (PA0)
- new net TIM5_CH1_2: JP2.10, U6.8 (PA0)
- new net TIM5_CH2_1: JP3.1, U1.9 (PA1)
- new net TIM5_CH2_2: JP3.7, U6.9 (PA1)
- new net TIM5_CH3_1: JP3.4, U1.10 (PA2)
- new net TIM5_CH3_2: JP3.10, U6.10 (PA2)
- new net TIM8_CH2N_1: JP1.1, U1.16 (PB0)
- new net TIM8_CH2N_2: JP2.1, U6.16 (PB0)
- new net TIM8_CH3N_1: JP1.4, U1.17 (PB1)
- new net TIM8_CH3N_2: JP2.4, U6.17 (PB1)
- new net USB2_CONN_D+: J8.3 (D+), U8.3 (I/O2)
- new net USB2_CONN_D-: J8.2 (D-), U8.1 (I/O1)
- new net USB2_D+: U6.34 (PA12), U8.4 (I/O2)
- new net USB2_D-: U6.33 (PA11), U8.6 (I/O1)
- no-connect marks 53 -> 39
Other:
- note added: "MCU 1:\n- 2x CAN Bus\n- BNO055\n\nMCU 2:\n- 2x CAN Bus"
- note added: "Q: These are tied differently... why?"
- note added: "Q: What does CH_N mean?\nAre these using the timers correctly?"
- moved on the sheet: C3

Commit message: Began board layout
Parts:
- added H1, H2, H3, H4: MountingHole_Pad, MountingHole:MountingHole_2.7mm_M2.5_DIN965, symbol Mechanical:MountingHole_Pad
- C19, C20, C21, C22, C24: footprint Capacitor_SMD:C_0402_1005Metric -> Capacitor_SMD:C_1206_3216Metric
- J1, J2, J3, J4: footprint Connector_JST:JST_PH_B4B-PH-K_1x04_P2.00mm_Vertical -> Connector_JST:JST_PH_B3B-PH-K_1x03_P2.00mm_Vertical
- renumbered 11 to 111
Connections:
- net GND: now also H1.1, H2.1, H3.1, H4.1
Changed lines of the file:
@@
 F 0 "J1" H 7605 1517 50  0000 L CNN
 F 1 "CAN 1 Conn" H 7605 1426 50  0000 L CNN
-F 2 "Connector_JST:JST_PH_B4B-PH-K_1x04_P2.00mm_Vertical" H 7525 1475 50  0001 C CNN
+F 2 "Connector_JST:JST_PH_B3B-PH-K_1x03_P2.00mm_Vertical" H 7525 1475 50  0001 C CNN
 F 3 "~" H 7525 1475 50  0001 C CNN
 	1    7525 1475
@@
 F 0 "J3" H 7605 3142 50  0000 L CNN
 F 1 "CAN 2 Conn" H 7605 3051 50  0000 L CNN
-F 2 "Connector_JST:JST_PH_B4B-PH-K_1x04_P2.00mm_Vertical" H 7525 3100 50  0001 C CNN
+F 2 "Connector_JST:JST_PH_B3B-PH-K_1x03_P2.00mm_Vertical" H 7525 3100 50  0001 C CNN
 F 3 "~" H 7525 3100 50  0001 C CNN
 	1    7525 3100
@@
 F 0 "J2" H 15680 1517 50  0000 L CNN
 F 1 "CAN 3 Conn" H 15680 1426 50  0000 L CNN
-F 2 "Connector_JST:JST_PH_B4B-PH-K_1x04_P2.00mm_Vertical" H 15600 1475 50  0001 C CNN
+F 2 "Connector_JST:JST_PH_B3B-PH-K_1x03_P2.00mm_Vertical" H 15600 1475 50  0001 C CNN
 F 3 "~" H 15600 1475 50  0001 C CNN
 	1    15600 1475
@@
 F 0 "C21" H 9792 7971 50  0000 L CNN
 F 1 "0.1uF 50V" H 9792 7880 50  0000 L CNN
-F 2 "Capacitor_SMD:C_0402_1005Metric" H 9700 7925 50  0001 C CNN
+F 2 "Capacitor_SMD:C_1206_3216Metric" H 9700 7925 50  0001 C CNN
 F 3 "~" H 9700 7925 50  0001 C CNN
 	1    9700 7925
@@
 F 0 "C20" H 9242 7971 50  0000 L CNN
 F 1 "0.1uF 50V" H 9242 7880 50  0000 L CNN
-F 2 "Capacitor_SMD:C_0402_1005Metric" H 9150 7925 50  0001 C CNN
+F 2 "Capacitor_SMD:C_1206_3216Metric" H 9150 7925 50  0001 C CNN
 F 3 "~" H 9150 7925 50  0001 C CNN
 	1    9150 7925
@@
 F 0 "C19" H 8692 7971 50  0000 L CNN
 F 1 "0.1uF 50V" H 8692 7880 50  0000 L CNN
-F 2 "Capacitor_SMD:C_0402_1005Metric" H 8600 7925 50  0001 C CNN
+F 2 "Capacitor_SMD:C_1206_3216Metric" H 8600 7925 50  0001 C CNN
 F 3 "~" H 8600 7925 50  0001 C CNN
 	1    8600 7925
@@
 $EndComp
 $Comp
-L xt30:XT30 11
+L xt30:XT30 111
 U 1 1 604C6C18
 P 6675 7625
-F 0 "11" H 6725 7675 50  0001 C CNN
+F 0 "111" H 6725 7675 50  0001 C CNN
 F 1 "XT30" H 6675 7625 50  0001 C CNN
 F 2 "helios_kicad_lib:XT30P" H 6675 7625 50  0001 C CNN
@@
 F 0 "C22" V 9371 8800 50  0000 C CNN
 F 1 "0.1uF 50V" V 9462 8800 50  0000 C CNN
-F 2 "Capacitor_SMD:C_0402_1005Metric" H 9600 8800 50  0001 C CNN
+F 2 "Capacitor_SMD:C_1206_3216Metric" H 9600 8800 50  0001 C CNN
 F 3 "~" H 9600 8800 50  0001 C CNN
 	1    9600 8800
@@
 F 0 "C24" H 9642 9746 50  0000 L CNN
 F 1 "10uF" H 9642 9655 50  0000 L CNN
-F 2 "Capacitor_SMD:C_0402_1005Metric" H 9550 9700 50  0001 C CNN
+F 2 "Capacitor_SMD:C_1206_3216Metric" H 9550 9700 50  0001 C CNN
 F 3 "~" H 9550 9700 50  0001 C CNN
 	1    9550 9700
@@
 F 0 "J4" H 15680 3142 50  0000 L CNN
 F 1 "CAN 4 Conn" H 15680 3051 50  0000 L CNN
-F 2 "Connector_JST:JST_PH_B4B-PH-K_1x04_P2.00mm_Vertical" H 15600 3100 50  0001 C CNN
+F 2 "Connector_JST:JST_PH_B3B-PH-K_1x03_P2.00mm_Vertical" H 15600 3100 50  0001 C CNN
 F 3 "~" H 15600 3100 50  0001 C CNN
 	1    15600 3100
@@
 Text GLabel 15725 9175 0    50   Input ~ 0
 TIM5_CH2_2
+$Comp
+L Mechanical:MountingHole_Pad H1
+U 1 1 61432AF7
+P 875 10400
+F 0 "H1" V 829 10550 50  0000 L CNN
+F 1 "MountingHole_Pad" V 920 10550 50  0000 L CNN
+F 2 "MountingHole:MountingHole_2.7mm_M2.5_DIN965" H 875 10400 50  0001 C CNN
+F 3 "~" H 875 10400 50  0001 C CNN
+	1    875  10400
+	0    1    1    0
+$EndComp
+$Comp
+L Mechanical:MountingHole_Pad H2
+U 1 1 614338CF
+P 875 10575
+F 0 "H2" V 829 10725 50  0000 L CNN
+F 1 "MountingHole_Pad" V 920 10725 50  0000 L CNN
+F 2 "MountingHole:MountingHole_2.7mm_M2.5_DIN965" H 875 10575 50  0001 C CNN
+F 3 "~" H 875 10575 50  0001 C CNN
+	1    875  10575
+	0    1    1    0
+$EndComp
+$Comp
+L Mechanical:MountingHole_Pad H3
+U 1 1 61433BC1
+P 875 10750
+F 0 "H3" V 829 10900 50  0000 L CNN
+F 1 "MountingHole_Pad" V 920 10900 50  0000 L CNN
+F 2 "MountingHole:MountingHole_2.7mm_M2.5_DIN965" H 875 10750 50  0001 C CNN
+F 3 "~" H 875 10750 50  0001 C CNN
+	1    875  10750
+	0    1    1    0
+$EndComp
+$Comp
+L Mechanical:MountingHole_Pad H4
+U 1 1 61433D9B
+P 875 10925
+F 0 "H4" V 829 11075 50  0000 L CNN
+F 1 "MountingHole_Pad" V 920 11075 50  0000 L CNN
+F 2 "MountingHole:MountingHole_2.7mm_M2.5_DIN965" H 875 10925 50  0001 C CNN
+F 3 "~" H 875 10925 50  0001 C CNN
+	1    875  10925
+	0    1    1    0
+$EndComp
+$Comp
+L power:GND #PWR0187
+U 1 1 61433F71
+P 775 10925
+F 0 "#PWR0187" H 775 10675 50  0001 C CNN
+F 1 "GND" H 780 10752 50  0000 C CNN
+F 2 "" H 775 10925 50  0001 C CNN
+F 3 "" H 775 10925 50  0001 C CNN
+	1    775  10925
+	1    0    0    -1
+$EndComp
+Wire Wire Line
+	775  10400 775  10575
+Connection ~ 775  10925
+Connection ~ 775  10575
+Wire Wire Line
+	775  10575 775  10750
+Connection ~ 775  10750
+Wire Wire Line
+	775  10750 775  10925
 $EndSCHEMATC

Commit message: Finished routing
Parts:
- added J9: Power Breakout, helios_kicad_lib:Eagle_1X03, symbol Connector_Generic:Conn_01x03
- H1, H2, H3, H4: footprint MountingHole:MountingHole_2.7mm_M2.5_DIN965 -> MountingHole:MountingHole_2.7mm_M2.5_DIN965_Pad
- J14: footprint Connector_PinHeader_2.54mm:PinHeader_1x03_P2.54mm_Vertical -> helios_kicad_lib:Eagle_1X03
- J22: footprint Connector_PinHeader_2.54mm:PinHeader_1x03_P2.54mm_Vertical -> Connector_PinHeader_2.54mm:PinHeader_1x04_P2.54mm_Vertical
- renumbered 111 to 1111
Connections:
- net SWDI_2 is gone; now on net SWDIO_2: J6.3 (Pin_3)
- net +3V3: now also J9.3 (Pin_3)
- net GND: now also U1.35 (VSS), U1.47 (VSS), J9.2 (Pin_2)
- net LED_1: now also U1.41 (PB4); no longer U1.5 (PF0-OSC_IN)
- net LED_2: now also U1.42 (PB5); no longer U1.6 (PF1-OSC_OUT)
- net LED_3: now also U6.41 (PB4); no longer U6.5 (PF0-OSC_IN)
- net LED_4: now also U6.42 (PB5); no longer U6.6 (PF1-OSC_OUT)
- net TIM20_CH1_1: now also JP3.7; no longer JP1.7
- net TIM20_CH1_2: now also JP2.1; no longer JP2.7
- net TIM5_CH1_2: now also JP3.4; no longer JP2.10
- net TIM5_CH2_1: now also JP1.7; no longer JP3.1
- net TIM5_CH2_2: now also JP3.1; no longer JP3.7
- net TIM5_CH3_1: now also JP1.4; no longer JP3.4
- net TIM5_CH3_2: now also JP2.10; no longer JP3.10
- net TIM8_CH2N_2: now also JP2.7; no longer JP2.1
- net TIM8_CH3N_1: now also JP3.10; no longer JP1.4
- net POWER_IN: now reaches 1111.+, F1.1, U9.+
- net POWER_IN: now also J9.1 (Pin_1)
Changed lines of the file:
@@
 Wire Wire Line
 	6500 4525 6500 4450
-Text GLabel 4150 1500 2    50   Input ~ 0
+Text GLabel 1350 3200 0    50   Input ~ 0
 LED_1
-Text GLabel 4150 1600 2    50   Input ~ 0
+Text GLabel 1350 3300 0    50   Input ~ 0
 LED_2
 $Comp
@@
 F 0 "J14" H 1043 8125 50  0000 C CNN
 F 1 "Serial Breakout" H 1043 8216 50  0000 C CNN
-F 2 "Connector_PinHeader_2.54mm:PinHeader_1x03_P2.54mm_Vertical" H 1125 8450 50  0001 C CNN
+F 2 "helios_kicad_lib:Eagle_1X03" H 1125 8450 50  0001 C CNN
 F 3 "~" H 1125 8450 50  0001 C CNN
 	1    1125 8450
@@
 F 0 "J22" H 5105 9567 50  0000 L CNN
 F 1 "I2C Breakout" H 5105 9476 50  0000 L CNN
-F 2 "Connector_PinHeader_2.54mm:PinHeader_1x03_P2.54mm_Vertical" H 5025 9575 50  0001 C CNN
+F 2 "Connector_PinHeader_2.54mm:PinHeader_1x04_P2.54mm_Vertical" H 5025 9575 50  0001 C CNN
 F 3 "~" H 5025 9575 50  0001 C CNN
 	1    5025 9575
@@
 SWO_2
 Text GLabel 9775 6525 0    50   Input ~ 0
-SWDI_2
+SWDIO_2
 Text GLabel 9775 6625 0    50   Input ~ 0
 SWCLK_2
@@
 Wire Wire Line
 	14575 4525 14575 4450
-Text GLabel 12225 1500 2    50   Input ~ 0
+Text GLabel 9425 3200 0    50   Input ~ 0
 LED_3
-Text GLabel 12225 1600 2    50   Input ~ 0
+Text GLabel 9425 3300 0    50   Input ~ 0
 LED_4
 $Comp
@@
 NoConn ~ 1350 2100
 NoConn ~ 1350 2600
-NoConn ~ 1350 3200
-NoConn ~ 1350 3300
 NoConn ~ 1350 3400
 NoConn ~ 1350 3500
@@
 NoConn ~ 1350 4000
 NoConn ~ 1350 4300
-NoConn ~ 9425 3200
-NoConn ~ 9425 3300
 NoConn ~ 9425 3400
 NoConn ~ 9425 3500
@@
 $EndComp
 $Comp
-L xt30:XT30 111
+L xt30:XT30 1111
 U 1 1 604C6C18
 P 6675 7625
-F 0 "111" H 6725 7675 50  0001 C CNN
+F 0 "1111" H 6725 7675 50  0001 C CNN
 F 1 "XT30" H 6675 7625 50  0001 C CNN
 F 2 "helios_kicad_lib:XT30P" H 6675 7625 50  0001 C CNN
@@
 $EndComp
 Wire Wire Line
-	2950 4975 2950 5375
-Wire Wire Line
 	1350 5175 1350 5075
 Wire Wire Line
@@
 Text GLabel 12850 8375 0    50   Input ~ 0
 TIM8_CH2N_1
-Text GLabel 12850 8775 0    50   Input ~ 0
+Text GLabel 15725 9575 0    50   Input ~ 0
 TIM8_CH3N_1
-Text GLabel 12850 9175 0    50   Input ~ 0
+Text GLabel 15725 9175 0    50   Input ~ 0
 TIM20_CH1_1
 Text GLabel 12850 9575 0    50   Input ~ 0
@@
 Connection ~ 14825 9775
 Connection ~ 14925 8475
-Text GLabel 14275 8375 0    50   Input ~ 0
+Text GLabel 14275 9175 0    50   Input ~ 0
 TIM8_CH2N_2
 Text GLabel 14275 8775 0    50   Input ~ 0
 TIM8_CH3N_2
-Text GLabel 14275 9175 0    50   Input ~ 0
+Text GLabel 14275 8375 0    50   Input ~ 0
 TIM20_CH1_2
-Text GLabel 14275 9575 0    50   Input ~ 0
+Text GLabel 15725 8775 0    50   Input ~ 0
 TIM5_CH1_2
 Wire Wire Line
@@
 Connection ~ 16275 9775
 Connection ~ 16375 8475
-Text GLabel 15725 9575 0    50   Input ~ 0
+Text GLabel 14275 9575 0    50   Input ~ 0
 TIM5_CH3_2
 Wire Wire Line
@@
 Wire Wire Line
 	15975 8775 15725 8775
+Text GLabel 12850 9175 0    50   Input ~ 0
+TIM5_CH2_1
+Text GLabel 12850 8775 0    50   Input ~ 0
+TIM5_CH3_1
 Text GLabel 15725 8375 0    50   Input ~ 0
-TIM5_CH2_1
-Text GLabel 15725 8775 0    50   Input ~ 0
-TIM5_CH3_1
-Text GLabel 15725 9175 0    50   Input ~ 0
 TIM5_CH2_2
 $Comp
@@
 F 0 "H1" V 829 10550 50  0000 L CNN
 F 1 "MountingHole_Pad" V 920 10550 50  0000 L CNN
-F 2 "MountingHole:MountingHole_2.7mm_M2.5_DIN965" H 875 10400 50  0001 C CNN
+F 2 "MountingHole:MountingHole_2.7mm_M2.5_DIN965_Pad" H 875 10400 50  0001 C CNN
 F 3 "~" H 875 10400 50  0001 C CNN
 	1    875  10400
@@
 F 0 "H2" V 829 10725 50  0000 L CNN
 F 1 "MountingHole_Pad" V 920 10725 50  0000 L CNN
-F 2 "MountingHole:MountingHole_2.7mm_M2.5_DIN965" H 875 10575 50  0001 C CNN
+F 2 "MountingHole:MountingHole_2.7mm_M2.5_DIN965_Pad" H 875 10575 50  0001 C CNN
 F 3 "~" H 875 10575 50  0001 C CNN
 	1    875  10575
@@
 F 0 "H3" V 829 10900 50  0000 L CNN
 F 1 "MountingHole_Pad" V 920 10900 50  0000 L CNN
-F 2 "MountingHole:MountingHole_2.7mm_M2.5_DIN965" H 875 10750 50  0001 C CNN
+F 2 "MountingHole:MountingHole_2.7mm_M2.5_DIN965_Pad" H 875 10750 50  0001 C CNN
 F 3 "~" H 875 10750 50  0001 C CNN
 	1    875  10750
@@
 F 0 "H4" V 829 11075 50  0000 L CNN
 F 1 "MountingHole_Pad" V 920 11075 50  0000 L CNN
-F 2 "MountingHole:MountingHole_2.7mm_M2.5_DIN965" H 875 10925 50  0001 C CNN
+F 2 "MountingHole:MountingHole_2.7mm_M2.5_DIN965_Pad" H 875 10925 50  0001 C CNN
 F 3 "~" H 875 10925 50  0001 C CNN
 	1    875  10925
@@
 Wire Wire Line
 	775  10750 775  10925
+Wire Wire Line
+	2950 4975 2950 5075
+Connection ~ 2950 5375
+Connection ~ 2950 5075
+Wire Wire Line
+	2950 5075 2950 5175
+Connection ~ 2950 5175
+Wire Wire Line
+	2950 5175 2950 5375
+$Comp
+L Connector_Generic:Conn_01x03 J9
+U 1 1 617721DA
+P 5025 8800
+F 0 "J9" H 5105 8842 50  0000 L CNN
+F 1 "Power Breakout" H 5105 8751 50  0000 L CNN
+F 2 "helios_kicad_lib:Eagle_1X03" H 5025 8800 50  0001 C CNN
+F 3 "~" H 5025 8800 50  0001 C CNN
+	1    5025 8800
+	1    0    0    -1
+$EndComp
+Text GLabel 7775 7825 3    50   Input ~ 0
+POWER_IN
+Text GLabel 4825 8700 0    50   Input ~ 0
+POWER_IN
+$Comp
+L power:GND #PWR0188
+U 1 1 61781F26
+P 4500 8800
+F 0 "#PWR0188" H 4500 8550 50  0001 C CNN
+F 1 "GND" H 4505 8627 50  0000 C CNN
+F 2 "" H 4500 8800 50  0001 C CNN
+F 3 "" H 4500 8800 50  0001 C CNN
+	1    4500 8800
+	1    0    0    -1
+$EndComp
+$Comp
+L power:+3V3 #PWR0189
+U 1 1 617911F6
+P 4725 9025
+F 0 "#PWR0189" H 4725 8875 50  0001 C CNN
+F 1 "+3V3" H 4725 9200 50  0000 C CNN
+F 2 "" H 4725 9025 50  0001 C CNN
+F 3 "" H 4725 9025 50  0001 C CNN
+	1    4725 9025
+	1    0    0    -1
+$EndComp
+Wire Wire Line
+	4500 8800 4825 8800
+Wire Wire Line
+	4725 9025 4825 9025
+Wire Wire Line
+	4825 9025 4825 8900
+NoConn ~ 4150 1500
+NoConn ~ 4150 1600
+NoConn ~ 12225 1500
+NoConn ~ 12225 1600
 $EndSCHEMATC

Commit message: Updated device addressing, added layout picture
Connections:
- net +3V3: no longer U6.3 (PC14-OSC32_IN)
- net GND: now also U6.3 (PC14-OSC32_IN)
Other:
- note removed: "MCU 1:\n- 2x CAN Bus\n- BNO055\n\nMCU 2:\n- 2x CAN Bus"
- note removed: "Q: These are tied differently... why?"
- note removed: "Q: What does CH_N mean?\nAre these using the timers correctly?"
Changed lines of the file:
@@
 	1    0    0    -1
 $EndComp
-Text Notes 3875 800  0    50   ~ 0
-Q: These are tied differently... why?
 $Comp
 L power:+3V3 #PWR0138
@@
 Text GLabel 4825 9775 0    50   Input ~ 0
 I2C2_SCL
-Text Notes 7825 -225 0    100  ~ 0
-MCU 1:\n- 2x CAN Bus\n- BNO055\n\nMCU 2:\n- 2x CAN Bus
 Text GLabel 3450 9750 2    50   Input ~ 0
 SPI0_SCK
@@
 Text GLabel 1350 3000 0    50   Input ~ 0
 TIM20_CH1_1
-Text Notes -1475 2875 0    50   ~ 0
-Q: What does CH_N mean?\nAre these using the timers correctly?
 NoConn ~ 2825 6975
 NoConn ~ 3225 6775
@@
 Wire Wire Line
 	11025 5175 11025 5075
-$Comp
-L power:+3V3 #PWR0180
-U 1 1 60DC8EF3
-P 12600 1200
-F 0 "#PWR0180" H 12600 1050 50  0001 C CNN
-F 1 "+3V3" H 12615 1373 50  0000 C CNN
-F 2 "" H 12600 1200 50  0001 C CNN
-F 3 "" H 12600 1200 50  0001 C CNN
-	1    12600 1200
-	1    0    0    -1
-$EndComp
 $Comp
 L power:+3V3 #PWR0181
@@
 NoConn ~ 12225 1500
 NoConn ~ 12225 1600
+Wire Wire Line
+	12600 1200 12600 1300
+Connection ~ 12600 1300
 $EndSCHEMATC
